Commit message: Modele urdf visuel

File: ws_ros/src/urdf_tutorial_zo/urdf/project.urdf (robot description, URDF)
Before this commit: robot sous_marin, 7 links, 6 joints
Joints:
- removed joint base_to_avant_droit
- removed joint base_to_avant_gauche
- removed joint base_to_bas
- removed joint base_to_haut
- removed joint base_to_left
- removed joint base_to_right
- added joint bras_arriere_bas_joint: type revolute, parent base_link, child panel_bas, origin xyz=0.0 1.4 0.055 rpy=0.0 1.57075 0.0, axis 1 0 0, limit lower=-0.548 upper=0.548 effort=1000.0 velocity=0.5
- added joint bras_arriere_droit_joint: type revolute, parent base_link, child panel_right, origin xyz=-0.095 1.4 0.15, axis 1 0 0, limit lower=-0.548 upper=0.548 effort=1000.0 velocity=0.5
- added joint bras_arriere_gauche_joint: type revolute, parent base_link, child panel_left, origin xyz=0.095 1.4 0.15, axis 1 0 0, limit lower=-0.548 upper=0.548 effort=1000.0 velocity=0.5
- added joint bras_arriere_haut_joint: type revolute, parent base_link, child panel_haut, origin xyz=0.0 1.4 0.24 rpy=0.0 1.57075 0.0, axis 1 0 0, limit lower=-0.548 upper=0.548 effort=1000.0 velocity=0.5
- added joint bras_avant_droit_joint: type revolute, parent base_link, child panel_avant_droit, origin xyz=-0.115 0.177 0.181 rpy=0 0.0 0, axis 1 0 0, limit lower=-0.548 upper=0.548 effort=1000.0 velocity=0.5
- added joint bras_avant_gauche_joint: type revolute, parent base_link, child panel_avant_gauche, origin xyz=0.115 0.177 0.181 rpy=0 3.14 0, axis 1 0 0, limit lower=-0.548 upper=0.548 effort=1000.0 velocity=0.5

Commit message: modification de l'urdf avec xacro

File: ws_ros/src/urdf_tutorial_zo/urdf/project.urdf (robot description, URDF)
Before this commit: robot sous_marin, 7 links, 6 joints
Links:
- link base_link: mass None -> 50.0; geometry collision mesh filename=package://urdf_tutorial_zo/meshes/coque_solide.dae; visual mesh filename=package://urdf_tutorial_zo/meshes/coque_solide.dae
Joints:
- joint bras_arriere_droit_joint: origin xyz=-0.095 1.4 0.15 -> xyz=-0.095 1.4 0.15 rpy=0 0.0 0
- joint bras_arriere_gauche_joint: origin xyz=0.095 1.4 0.15 -> xyz=0.095 1.4 0.15 rpy=0 3.14 0
